File: JEGGER_s-link.kicad_pcb (KiCad board)
At the start: 2 copper layers, 37.6 x 16.1 mm, 39 parts, among them J1 USB, J2 TC, J3 PINH, J4 RX, J5 TX, P1 STM, U1 USBLC6-4, U2 MCP1700T-3302E/TT, U3 STM32F103CBTx, Y1 8Mhz

Commit message: layout done
Parts:
- removed C10, C11: 0.1µ, otter:C_0402
- removed G***: LOGO, otter:jegger_233
- removed G***: LOGO, otter:kicad_designer_84
- removed P1: STM, otter:TC2030
- removed R15, R16, R17, R19, R20: 5k1, otter:R_0402
- added C1: 1u, Capacitor_SMD:C_0402_1005Metric, F.Cu at (110.7, 52.4)
- added F1: 500mA, Fuse:Fuse_0603_1608Metric, F.Cu at (110.4, 53.7)
- added R12: 5K1, Resistor_SMD:R_0402_1005Metric, F.Cu at (120.3, 60.5)
- added R14: 1K5, Resistor_SMD:R_0402_1005Metric, F.Cu at (110.5, 58.2)
- added R6: 5K1, Resistor_SMD:R_0402_1005Metric, F.Cu at (109.5, 58.2)
- added R7: 5K1, Resistor_SMD:R_0402_1005Metric, F.Cu at (110.0, 59.7)
- added R8: 100R, Resistor_SMD:R_0402_1005Metric, F.Cu at (126.1, 59.0)
- C2: value 0.1µ -> 1u; footprint otter:C_0402 -> Capacitor_SMD:C_0402_1005Metric
- C3: value 0.1µ -> 22p; footprint otter:C_0402 -> Capacitor_SMD:C_0402_1005Metric
- C4: footprint otter:C_0402 -> Capacitor_SMD:C_0402_1005Metric
- C5: value 22p -> 100n; footprint otter:C_0402 -> Capacitor_SMD:C_0402_1005Metric
- C6, C7: value 10µ -> 100n; footprint otter:C_0402 -> Capacitor_SMD:C_0402_1005Metric
- C8: value 0.1µ -> 100n; footprint otter:C_0402 -> Capacitor_SMD:C_0402_1005Metric
- D1: value PWR -> GREEN
- D2: value BAT60JFILM -> RED; footprint Diode_SMD:D_SOD-323 -> LED_SMD:LED_0603_1608Metric
- D3: value GREEN -> BAT60JFILM; footprint LED_SMD:LED_0603_1608Metric -> Diode_SMD:D_SOD-323
- D4: value RED -> PWR
- J1: footprint otter:USB-C 16Pin -> josh-connectors:USB_C_U262-161N-4BVC11
- J2: value TC -> Tag-Connect; footprint otter:IDC-Header_2x03_P2.54mm_Vertical_center -> Connector_IDC:IDC-Header_2x03_P2.54mm_Vertical
- J3: value PINH -> STM_DEBUG; footprint otter:PinHeader_1x06_P2.54mm_Vertical_center -> josh-connectors:STM_5_PIN_SMD_PROG; moved to B.Cu
- J4: value RX -> OUT; footprint TestPoint:TestPoint_Pad_1.0x1.0mm -> josh-connectors:STM_6_PIN_THT_Staggered; moved to F.Cu
- J5: value TX -> STLINK_UART; footprint TestPoint:TestPoint_Pad_1.0x1.0mm -> josh-connectors:UART_3_PIN_SMD_PROG
- R1: value 5k1 -> 10K; footprint otter:R_0402 -> Resistor_SMD:R_0402_1005Metric
- R10, R2, R3, R9: value 5k1 -> 5K1; footprint otter:R_0402 -> Resistor_SMD:R_0402_1005Metric
- R11: value 1k5 -> 5K1; footprint otter:R_0402 -> Resistor_SMD:R_0402_1005Metric
- R13, R5: value 100 -> 5K1; footprint otter:R_0402 -> Resistor_SMD:R_0402_1005Metric
- R4: value 10k -> 100R; footprint otter:R_0402 -> Resistor_SMD:R_0402_1005Metric
- U1: value USBLC6-4 -> USBLC6-2P6; footprint Package_TO_SOT_SMD:SOT-23-6 -> Package_TO_SOT_SMD:SOT-666
- U2: value MCP1700T-3302E/TT -> AP2112K-3.3; footprint Package_TO_SOT_SMD:SOT-23 -> Package_TO_SOT_SMD:SOT-23-5
- U3: footprint otter:LQFP-48_7x7mm_P0.5mm -> Package_QFP:LQFP-48_7x7mm_P0.5mm
- moved J5 60.9 mm to (134.5, 47.5), turned to 90 degrees
- moved C8 57.3 mm to (115.0, 48.6), turned to 180 degrees
- moved R5 57.0 mm to (113.1, 50.0), turned to 180 degrees
- moved C5 56.2 mm to (122.8, 50.2), turned to 180 degrees
- moved R2 55.8 mm to (122.8, 49.2), turned to 0 degrees
- moved D2 54.9 mm to (125.4, 48.3), turned to 180 degrees
- moved C4 53.0 mm to (124.7, 51.6), turned to 0 degrees
- moved Y1 51.2 mm to (125.1, 54.3), turned to 90 degrees
- moved R3 50.6 mm to (122.8, 48.2), turned to 180 degrees
- moved J4 49.7 mm to (138.8, 60.6), turned to 180 degrees
- moved C3 49.0 mm to (124.7, 57.0), turned to 0 degrees
- moved C2 48.5 mm to (113.1, 48.6), turned to 0 degrees
- moved D1 48.0 mm to (125.4, 49.9), turned to 0 degrees
- moved D4 47.6 mm to (112.6, 60.0), turned to 0 degrees
- moved U2 45.9 mm to (110.2, 50.0), turned to 90 degrees
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Connections:
- C2 pad 1: VBUS -> +3V3
- C3 pad 1: +3V3 -> GND
- C3 pad 2: GND -> Net-(C3-Pad2)
- C4 pad 1: GND -> Net-(C4-Pad1)
- C4 pad 2: Net-(C4-Pad2) -> GND
- C5 pad 1: Net-(C5-Pad1) -> GND
- C5 pad 2: GND -> /STM_nRST
- C6 pad 1: VBUS -> GND
- C6 pad 2: GND -> +3V3
- C7 pad 1: +3V3 -> GND
- C7 pad 2: GND -> +3V3
- C8 pad 1: STM_NRST -> GND
- C8 pad 2: GND -> +3V3
- D2 pad 1: Net-(D2-Pad1) -> GND
- D2 pad 2: REF -> Net-(D2-Pad2)
- D3 pad 2: +3V3 -> /V_REF
- D4 pad 1: GND -> Net-(D4-Pad1)
- D4 pad 2: Net-(D4-Pad2) -> +3V3
- J1 pad A4: VBUS -> Net-(F1-Pad2)
- J1 pad A6: D+ -> /USB_D+
- J1 pad A7: D- -> /USB_D-
- J1 pad A8: Net-(J1-PadA8) -> (no net)
- J1 pad A9: VBUS -> Net-(F1-Pad2)
- J1 pad B4: VBUS -> Net-(F1-Pad2)
- J1 pad B6: D+ -> /USB_D+
- J1 pad B7: D- -> /USB_D-
- J1 pad B8: Net-(J1-PadB8) -> (no net)
- J1 pad B9: VBUS -> Net-(F1-Pad2)
- J2 pad 1: REF -> /V_REF
- J2 pad 2: T_JTMS -> /T_JTMS
- J2 pad 3: T_NRST -> /T_nRST
- J2 pad 4: T_JTCK -> /T_JTCK
- J2 pad 6: T_SWO -> /T_SWO
- J3 pad 1: REF -> +3V3
- J3 pad 2: T_JTCK -> /STM_JTCK
- J3 pad 4: T_JTMS -> /STM_JTMS
- J3 pad 5: T_NRST -> /STM_nRST
- J4 pad 1: STLINK_RX -> /V_REF
- J5 pad 1: STLINK_TX -> GND
- R1 pad 2: Net-(J1-PadA5) -> /V_REF
- R10 pad 1: Net-(D4-Pad2) -> Net-(R10-Pad1)
- R10 pad 2: LED_STLINK -> GND
- R11 pad 1: +3V3 -> Net-(R11-Pad1)
- R11 pad 2: D+ -> GND
- R13 pad 1: T_JTMS -> /A_IN
- R13 pad 2: T_SWDIO_IN -> GND
- R2 pad 1: GND -> /LED_STLINK
- R2 pad 2: Net-(J1-PadB5) -> Net-(D1-Pad1)
- R3 pad 1: Net-(D1-Pad1) -> Net-(D2-Pad2)
- R3 pad 2: GND -> /LED_STLINK
- R4 pad 1: GND -> Net-(D3-Pad1)
- R4 pad 2: REF -> /A_IN
- R5 pad 1: Net-(D2-Pad1) -> GND
- R5 pad 2: AIN_1 -> Net-(J1-PadA5)
- R9 pad 1: LED_STLINK -> Net-(R9-Pad1)
- R9 pad 2: Net-(D3-Pad1) -> GND
- U1 pad 1: D- -> /USB_D-
- U1 pad 3: Net-(U1-Pad3) -> /USB_D+
- U1 pad 4: Net-(U1-Pad4) -> /D+
- U1 pad 6: D+ -> /D-
- U2 pad 1: GND -> VBUS
- U2 pad 2: +3V3 -> GND
- U3 pad 10: AIN_1 -> /A_IN
- U3 pad 11: Net-(U3-Pad11) -> (no net)
- U3 pad 12: STLINK_TX -> /STLINK_TX
- U3 pad 13: STLINK_RX -> /STLINK_RX
- U3 pad 14: Net-(U3-Pad14) -> (no net)
- U3 pad 15: T_JTCK -> /T_JTCK
- U3 pad 16: T_JTDO -> (no net)
- U3 pad 17: T_JTDI -> (no net)
- U3 pad 18: T_NRST -> /T_nRST
- U3 pad 19: T_JRST -> (no net)
- U3 pad 2: Net-(R15-Pad1) -> Net-(R9-Pad1)
- U3 pad 21: Net-(U3-Pad21) -> (no net)
- U3 pad 22: Net-(U3-Pad22) -> (no net)
- U3 pad 25: T_SWDIO_IN -> /T_SWDIO_IN
- U3 pad 26: T_JTCK -> /T_JTCK
- U3 pad 27: T_JTMS -> /T_JTMS
- U3 pad 28: PWR_EN -> (no net)
- U3 pad 29: Net-(U3-Pad29) -> (no net)
- U3 pad 3: Net-(R16-Pad1) -> Net-(R10-Pad1)
- U3 pad 30: LED_STLINK -> /LED_STLINK
- U3 pad 31: T_SWO -> /T_SWO
- U3 pad 32: D- -> /D-
- U3 pad 33: D+ -> /D+
- U3 pad 34: STM_JTMS -> /STM_JTMS
- U3 pad 37: STM_JTCK -> /STM_JTCK
- U3 pad 38: USB_RENUM -> (no net)
- U3 pad 4: Net-(U3-Pad4) -> (no net)
- U3 pad 40: Net-(U3-Pad40) -> (no net)
- U3 pad 41: Net-(U3-Pad41) -> (no net)
- U3 pad 42: Net-(U3-Pad42) -> (no net)
- U3 pad 43: Net-(U3-Pad43) -> (no net)
- U3 pad 44: Net-(R17-Pad1) -> Net-(R11-Pad1)
- U3 pad 45: Net-(U3-Pad45) -> (no net)
- U3 pad 46: Net-(U3-Pad46) -> (no net)
- U3 pad 5: Net-(C4-Pad2) -> Net-(C3-Pad2)
- U3 pad 6: Net-(C5-Pad1) -> Net-(C4-Pad1)
- U3 pad 7: STM_NRST -> /STM_nRST
- Y1 pad 1: Net-(C4-Pad2) -> Net-(C3-Pad2)
- Y1 pad 3: Net-(C5-Pad1) -> Net-(C4-Pad1)
Routing:
- net /T_JTCK: track 0.00 -> 35.8 mm, vias 0 -> 4
- net +3V3: track 52.9 -> 87.5 mm, vias 4 -> 6
- net /T_SWO: track 0.00 -> 33.8 mm, vias 0 -> 2
- net /T_JTMS: track 0.00 -> 32.0 mm, vias 0 -> 2
- net /T_nRST: track 0.00 -> 27.8 mm, vias 0 -> 2
- net /STM_nRST: track 0.00 -> 26.0 mm, vias 0 -> 3
- net T_JTCK: track 23.2 -> 0.00 mm, vias 2 -> 0
- net D+: track 22.5 -> 0.00 mm, vias 3 -> 0
- net /STM_JTMS: track 0.00 -> 21.9 mm, vias 0 -> 3
- net D-: track 19.4 -> 0.00 mm, vias 2 -> 0
- net /V_REF: track 0.00 -> 19.3 mm
- net T_SWO: track 19.3 -> 0.00 mm, vias 1 -> 0
- net T_JTMS: track 19.0 -> 0.00 mm
- net T_NRST: track 18.0 -> 0.00 mm, vias 2 -> 0
- net Net-(D3-Pad1): track 18.9 -> 1.29 mm, vias 2 -> 0
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Other:
- board size 37.6 x 16.1 mm -> 44.8 x 16.3 mm
- net class Default: via_drill 0.4 -> 0.3
- board text added: "3V3"
- board text added: "Original Design: @JanHenrikH Modifications: @_joshajohnson"
- board text added: "PWR"
- board text removed: "Design by: @JanHenrikH"

Commit message: added silk
Parts:
- added G***: LOGO, josh-connectors:kicad_designer_84, B.Cu at (126.3, 53.0)
- added G***: LOGO, josh-connectors:jegger_233, B.Cu at (112.5, 54.3)
Other:
- board text added: "Modified By: @_joshajohnson"
- board text added: "Original Design: @JanHenrikH"
- board text removed: "Original Design: @JanHenrikH Modifications: @_joshajohnson"
