File: JEGGER_s-link.sch (KiCad schematic (older format))
At the start: 37 parts, among them J1 USB, J2 TC, J3 PINH, J4 RX, J5 TX, P1 STM, U1 USBLC6-4, U2 MCP1700T-3302E/TT, U3 STM32F103CBTx, Y1 8Mhz

Commit message: changed schematic
Parts:
- removed C10, C11, C2, C3, C8: 0.1µ, otter:C_0402, symbol Device:C_Small
- removed C6, C7: 10µ, otter:C_0402, symbol Device:C_Small
- removed J4: RX, TestPoint:TestPoint_Pad_1.0x1.0mm, symbol Connector:Conn_01x01_Male
- removed J5: TX, TestPoint:TestPoint_Pad_1.0x1.0mm, symbol Connector:Conn_01x01_Male
- removed P1: STM, otter:TC2030, symbol otter:TC2030-CTX-Tag-Connect
- removed U2: MCP1700T-3302E/TT, Package_TO_SOT_SMD:SOT-23, symbol Regulator_Linear:MCP1700-3302E_SOT23
- added C1, C2: 1u, symbol Device:C
- added C5, C6, C7, C8: 100n, symbol Device:C
- added F1: 500mA, symbol Device:Polyfuse_Small
- added J?: STM_DEBUG, symbol Connector_Generic:Conn_01x05
- added J?: STLINK_UART, symbol Connector_Generic:Conn_01x02
- added U2: AP2112K-3.3, Package_TO_SOT_SMD:SOT-23-5, symbol Regulator_Linear:AP2112K-3.3
- D3: renamed from D2; symbol JEGGER_s-link-rescue:BAT60A-Diode -> JEGGER_s-link-rescue:BAT60A-Diode-JEGGER_s-link-rescue
- J2: value TC -> Tag-Connect
- J4: renamed from J3; value PINH -> OUT
- R1: renamed from R4; value 10k -> 10K
- R10: renamed from R16; value 5k1 -> 5K1
- R11: renamed from R17; value 5k1 -> 5K1
- R12: renamed from R19; value 5k1 -> 5K1
- R13: renamed from R20; value 5k1 -> 5K1
- R14: renamed from R11; value 1k5 -> 1K5
- R2: renamed from R9; value 5k1 -> 5K1
- R3: renamed from R10; value 5k1 -> 5K1
- R4: renamed from R5; value 100 -> 100R
- R5: renamed from R1; value 5k1 -> 5K1
- R6: renamed from R2; value 5k1 -> 5K1
- R7: renamed from R3; value 5k1 -> 5K1
- R8: renamed from R13; value 100 -> 100R
- R9: renamed from R15; value 5k1 -> 5K1
- U1: symbol otter:USBLC6-4 -> JEGGER_s-link-rescue:USBLC6-4-otter
- renumbered C4 to C3, C5 to C4, D3 to D1, D4 to D2, D1 to D4
Connections:
- net labels added: +3V3, A_IN, STM_nRST, T_nRST, USB_D+, USB_D-, V_REF
- net labels removed: AIN_1, REF, STM_NRST, T_NRST
- wire segments 73 -> 159
- no-connect marks 12 -> 14
Other:
- note added: "JTAG / SWD Out"
- note added: "Program STM32"
- moved on the sheet: C3, C4, D1, D2, D4, J1, J2, J4, R1, R10, R11, R12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

Commit message: layout done
Parts:
- removed J?: STLINK_UART, symbol Connector_Generic:Conn_01x02
- removed U1: USBLC6-4, Package_TO_SOT_SMD:SOT-23-6, symbol JEGGER_s-link-rescue:USBLC6-4-otter
- added J5: STLINK_UART, josh-connectors:UART_3_PIN_SMD_PROG, symbol Connector_Generic:Conn_01x03
- added U1: USBLC6-2P6, Package_TO_SOT_SMD:SOT-666, symbol Power_Protection:USBLC6-2P6
- C1, C2, C5, C6, C7, C8: footprint (none) -> Capacitor_SMD:C_0402_1005Metric
- C3, C4: footprint otter:C_0402 -> Capacitor_SMD:C_0402_1005Metric
- F1: footprint (none) -> Fuse:Fuse_0603_1608Metric
- J1: footprint otter:USB-C 16Pin -> josh-connectors:USB_C_U262-161N-4BVC11
- J2: footprint otter:IDC-Header_2x03_P2.54mm_Vertical_center -> Connector_IDC:IDC-Header_2x03_P2.54mm_Vertical
- J3: renamed from J?; footprint (none) -> josh-connectors:STM_5_PIN_SMD_PROG
- J4: footprint otter:PinHeader_1x06_P2.54mm_Vertical_center -> josh-connectors:STM_6_PIN_THT_Staggered
- R1, R10, R11, R12, R13, R14, R2, R3, R4, R5, R6, R7, R8, R9: footprint otter:R_0402 -> Resistor_SMD:R_0402_1005Metric
- U3: footprint otter:LQFP-48_7x7mm_P0.5mm -> Package_QFP:LQFP-48_7x7mm_P0.5mm
Connections:
- net D+: now also U1.4 (I/O2)
- net D-: now also U1.6 (I/O1)
- net GND: now also J5.1 (Pin_1), U1.2 (GND)
- net STLINK_RX: now also J5.2 (Pin_2)
- net STLINK_TX: now also J5.3 (Pin_3)
- net USB_D+: now also U1.3 (I/O2)
- net USB_D-: now also U1.1 (I/O1)
- net VBUS: now also U1.5 (VBUS)

Commit message: generated gerbers
Parts:
- J5: value STLINK_UART -> TGT_UART
Connections:
- net STLINK_RX renamed T_RX
- net STLINK_TX renamed T_TX
Other:
- moved on the sheet: J5
Changed lines of the file:
@@
 	6350 2250 6350 2550
 Text Label 7400 4150 2    50   ~ 0
-STLINK_RX
+T_RX
 Wire Wire Line
 	7400 4150 6950 4150
@@
 	6950 4050 7400 4050
 Text Label 7400 4050 2    50   ~ 0
-STLINK_TX
+T_TX
 Text Label 8950 3350 0    50   ~ 0
 V_REF
@@
 Text Label 5200 5050 0    50   ~ 0
 T_SWDIO_IN
-Wire Wire Line
-	5200 5050 5650 5050
-Text Label 4500 5250 0    50   ~ 0
-T_SWDIO_IN
-Wire Wire Line
-	4500 5250 4950 5250
 Text Label 7400 4450 2    50   ~ 0
 T_JTDO
@@
 JTAG / SWD Out
 $Comp
+L power:GND #PWR0103
+U 1 1 5F46D5AE
+P 1350 5800
+F 0 "#PWR0103" H 1350 5550 50  0001 C CNN
+F 1 "GND" H 1355 5627 50  0000 C CNN
+F 2 "" H 1350 5800 50  0001 C CNN
+F 3 "" H 1350 5800 50  0001 C CNN
+	1    1350 5800
+	1    0    0    -1
+$EndComp
+Wire Wire Line
+	1500 5750 1350 5750
+Wire Wire Line
+	1350 5750 1350 5800
+Wire Wire Line
+	1050 5650 1500 5650
+Wire Wire Line
+	1050 5550 1500 5550
+Text Label 1050 5550 0    50   ~ 0
+T_TX
+Text Label 1050 5650 0    50   ~ 0
+T_RX
+$Comp
+L Power_Protection:USBLC6-2P6 U1
+U 1 1 5F4B02DF
+P 3350 1750
+F 0 "U1" H 3100 2100 50  0000 C CNN
+F 1 "USBLC6-2P6" H 3650 2100 50  0000 C CNN
+F 2 "Package_TO_SOT_SMD:SOT-666" H 3350 1250 50  0001 C CNN
+F 3 "https://www.st.com/resource/en/datasheet/usblc6-2.pdf" H 3550 2100 50  0001 C CNN
+	1    3350 1750
+	1    0    0    -1
+$EndComp
+Wire Wire Line
+	3350 1300 3350 1350
+Connection ~ 6450 2550
+Connection ~ 6250 2550
+Wire Wire Line
+	6350 2550 6450 2550
+Wire Wire Line
+	6450 2550 6550 2550
+Wire Wire Line
+	6150 2550 6250 2550
+Wire Wire Line
+	6250 2550 6350 2550
+$Comp
 L MCU_ST_STM32F1:STM32F103CBTx U3
 U 1 1 5F43E051
@@
 	1    0    0    -1
 $EndComp
-Wire Wire Line
-	6250 2550 6350 2550
-Wire Wire Line
-	6450 2550 6550 2550
-$Comp
-L power:GND #PWR0103
-U 1 1 5F46D5AE
-P 1350 5750
-F 0 "#PWR0103" H 1350 5500 50  0001 C CNN
-F 1 "GND" H 1355 5577 50  0000 C CNN
-F 2 "" H 1350 5750 50  0001 C CNN
-F 3 "" H 1350 5750 50  0001 C CNN
-	1    1350 5750
-	1    0    0    -1
-$EndComp
-Wire Wire Line
-	1500 5700 1350 5700
-Wire Wire Line
-	1350 5700 1350 5750
-Wire Wire Line
-	1050 5600 1500 5600
-Wire Wire Line
-	1050 5500 1500 5500
-Text Label 1050 5500 0    50   ~ 0
-STLINK_TX
-Text Label 1050 5600 0    50   ~ 0
-STLINK_RX
 $Comp
 L Connector_Generic:Conn_01x03 J5
 U 1 1 5F46500A
-P 1700 5600
-F 0 "J5" H 1800 5550 50  0000 C CNN
-F 1 "STLINK_UART" H 2000 5650 50  0000 C CNN
-F 2 "josh-connectors:UART_3_PIN_SMD_PROG" H 1700 5600 50  0001 C CNN
-F 3 "~" H 1700 5600 50  0001 C CNN
-	1    1700 5600
+P 1700 5650
+F 0 "J5" H 1900 5600 50  0000 C CNN
+F 1 "TGT_UART" H 2000 5700 50  0000 C CNN
+F 2 "josh-connectors:UART_3_PIN_SMD_PROG" H 1700 5650 50  0001 C CNN
+F 3 "~" H 1700 5650 50  0001 C CNN
+	1    1700 5650
 	1    0    0    1
 $EndComp
-$Comp
-L Power_Protection:USBLC6-2P6 U1
-U 1 1 5F4B02DF
-P 3350 1750
-F 0 "U1" H 3100 2100 50  0000 C CNN
-F 1 "USBLC6-2P6" H 3650 2100 50  0000 C CNN
-F 2 "Package_TO_SOT_SMD:SOT-666" H 3350 1250 50  0001 C CNN
-F 3 "https://www.st.com/resource/en/datasheet/usblc6-2.pdf" H 3550 2100 50  0001 C CNN
-	1    3350 1750
-	1    0    0    -1
-$EndComp
-Wire Wire Line
-	3350 1300 3350 1350
-Wire Wire Line
-	6150 2550 6250 2550
-Connection ~ 6250 2550
-Wire Wire Line
-	6350 2550 6450 2550
-Connection ~ 6450 2550
+Wire Wire Line
+	4950 5250 4900 5250
+Wire Wire Line
+	4900 5250 4900 5050
+Wire Wire Line
+	4900 5050 5650 5050
 $EndSCHEMATC
